File: CRT Main PCB/CRT Driver.kicad_pcb (KiCad board)
At the start: 2 copper layers, 85 x 56 mm, 59 parts, among them J4 CRT, J5 TRANSFORMER, J6 XYZ SIGNAL IN, Q1 ZTX458, Q2 ZTX458, Q4 ZTX458, Q5 ZTX458, Q9 ZTX458, U1 TL082, U4 L78L05_TO92, U5 L79L05_SO8

Commit message: PCB changes
Parts:
- Q1, Q2, Q4, Q5, Q9, U4: footprint Package_TO_SOT_THT:TO-92_Inline -> Package_TO_SOT_THT:TO-92_Inline_Wide
- U5: value L79L05_SO8 -> L79L05_TO92; footprint Package_TO_SOT_THT:TO-92_Inline -> Package_TO_SOT_THT:TO-92_Inline_Wide
- moved C19 4.23 mm to (172.8, 73.6)
- moved R2 3.32 mm to (159.7, 93.0)
- moved Q5 2.82 mm to (160.9, 105.0), turned to 90 degrees
- moved Q1 2.74 mm to (154.2, 113.0), turned to 90 degrees
- moved Q2 2.52 mm to (160.9, 113.0), turned to 90 degrees
- moved Q4 2.31 mm to (154.2, 105.0), turned to 90 degrees
- moved U4 2.23 mm to (181.1, 74.2)
- moved U5 2.16 mm to (181.1, 80.0)
- moved C21 2.08 mm to (172.4, 81.8)
- renumbered 5V1 to 5V, ASTIG1 to ASTIG, FOCUS1 to FOCUS, INTENSITY1 to INTENSITY, XPOS1 to XPOS, XSIZE1 to XSIZE, YPOS1 to YPOS, YSIZE1 to YSIZE
Connections:
- 5V pad 2: HV CENTER -> 6.3V OPAMP A
- ASTIG pad 3: HV CENTER -> 6.3V OPAMP A
- C15 pad 2: HV CENTER -> 6.3V OPAMP A
- C18 pad 1: HV CENTER -> 6.3V OPAMP A
- C19 pad 1: HV CENTER -> 6.3V OPAMP A
- C20 pad 2: HV CENTER -> 6.3V OPAMP A
- C21 pad 2: HV CENTER -> 6.3V OPAMP A
- C22 pad 1: HV CENTER -> 6.3V OPAMP A
- C22 pad 2: Net-(D8-Pad2) -> Net-(C22-Pad2)
- D4 pad 1: HV CENTER -> 6.3V OPAMP A
- D8 pad 2: Net-(D8-Pad2) -> Net-(C22-Pad2)
- J5 pad 3: HV CENTER -> 6.3V OPAMP A
- J5 pad 6: HV CENTER -> 6.3V OPAMP A
- J6 pad 3: HV CENTER -> 6.3V OPAMP A
- Q9 pad 1: HV CENTER -> 6.3V OPAMP A
- R1 pad 1: HV CENTER -> 6.3V OPAMP A
- R10 pad 1: HV CENTER -> 6.3V OPAMP A
- R11 pad 2: HV CENTER -> 6.3V OPAMP A
- U4 pad 2: HV CENTER -> 6.3V OPAMP A
- U5 pad 1: -5V -> 6.3V OPAMP A
- U5 pad 2: Net-(D8-Pad2) -> Net-(C22-Pad2)
- U5 pad 3: Net-(D8-Pad2) -> -5V
- XSIZE pad 3: HV CENTER -> 6.3V OPAMP A
- YSIZE pad 3: HV CENTER -> 6.3V OPAMP A
Routing:
- net +5V: track 52.2 -> 147.4 mm, vias 0 -> 1
- net +HV: track 85.4 -> 119.3 mm, vias 0 -> 1
- net Net-(Q5-Pad2): track 20.2 -> 52.3 mm
- net Y2: track 6.40 -> 37.3 mm
- net Net-(Q1-Pad1): track 0.00 -> 27.7 mm
- net -5V: track 27.3 -> 0.17 mm
- net X2: track 11.3 -> 38.2 mm
- net Net-(C22-Pad2): track 0.00 -> 25.2 mm
- net Net-(Q5-Pad1): track 0.00 -> 24.2 mm
- net Net-(Q2-Pad2): track 4.77 -> 28.8 mm
- net Net-(R1-Pad2): track 0.00 -> 21.5 mm, vias 0 -> 1
- net Net-(C21-Pad1): track 24.2 -> 41.7 mm
- net Net-(R10-Pad2): track 12.3 -> 29.2 mm, vias 0 -> 1
- net Net-(Q4-Pad2): track 5.41 -> 21.3 mm
- net Net-(Q1-Pad2): track 0.00 -> 14.3 mm
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- added copper zone on F.Cu, net -5V
- added copper zone on B.Cu, net 6.3V OPAMP A
- removed copper zone on B.Cu, net HV CENTER
Other:
- board text added: "CGULA CRT DRIVER REV. 1.0"
- board text added: "FOCUS INTEN"
- board text added: "GND"
- board text added: "HEATER B HEATER A"
- board text added: "HVA | GND | HEATERA | HEATERB"
- board text added: "HVB | NC | 6.3PWRA | 6.3PWRB"
- board text added: "INPUT"
- board text added: "NC NC"
- board text added: "X1 X2"
- board text added: "Y1 Y2"
- board text added: "Z GND Y X"
- board text added: "ZGRID ASTIG"

Commit message: fixed errors
Parts:
- R11: value 4.7K -> 470K
- renumbered 5V to 5V1, ASTIG to ASTIG1, FOCUS to FOCUS1, INTENSITY to INTENSITY1, XPOS to XPOS1, XSIZE to XSIZE1, YPOS to YPOS1, YSIZE to YSIZE1
Other:
- board text added: "CGULA CRT DRIVER REV. 1.1"
- board text removed: "CGULA CRT DRIVER REV. 1.0"
Changed lines of the file:
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@@
     (property "Sheetname" "")
     (attr through_hole)
-    (fp_text reference "XSIZE" (at -2.1 4.2 unlocked) (layer "F.SilkS")
+    (fp_text reference "XSIZE1" (at -2.1 4.2 unlocked) (layer "F.SilkS")
       (effects (font (size 1 1) (thickness 0.15)))
     )
@@
     (property "Sheetname" "")
     (attr through_hole)
-    (fp_text reference "XPOS" (at -2.1 4.2 unlocked) (layer "F.SilkS")
+    (fp_text reference "XPOS1" (at -2.1 4.2 unlocked) (layer "F.SilkS")
       (effects (font (size 1 1) (thickness 0.15)))
     )
@@
       (effects (font (size 1 1) (thickness 0.15)))
     )
-    (fp_text user "K" (at 0 -2.1) (layer "F.SilkS")
-      (effects (font (size 1 1) (thickness 0.15)))
-    )
     (fp_text user "${REFERENCE}" (at 5.47 0) (layer "F.Fab")
       (effects (font (size 1 1) (thickness 0.15)))
@@
       (effects (font (size 1 1) (thickness 0.15)))
     )
-    (fp_text user "K" (at 0 -2.1 90) (layer "F.SilkS")
-      (effects (font (size 1 1) (thickness 0.15)))
-    )
     (fp_text user "${REFERENCE}" (at 5.47 0 90) (layer "F.Fab")
       (effects (font (size 1 1) (thickness 0.15)))
@@
     (property "Sheetname" "")
     (attr through_hole)
-    (fp_text reference "R2" (at 5.08 -2.37) (layer "F.SilkS")
+    (fp_text reference "R2" (at 5.17 1.52) (layer "F.SilkS")
       (effects (font (size 1 1) (thickness 0.15)))
     )
@@
     (property "Sheetname" "")
     (attr through_hole)
-    (fp_text reference "R6" (at 0.4 -2.6) (layer "F.SilkS")
+    (fp_text reference "R6" (at 5.33 1.65) (layer "F.SilkS")
       (effects (font (size 1 1) (thickness 0.15)))
     )
@@
     (property "Sheetname" "")
     (attr through_hole)
-    (fp_text reference "Q9" (at 2.54 -3.56) (layer "F.SilkS")
+    (fp_text reference "Q9" (at 2.54 -1.74) (layer "F.SilkS")
       (effects (font (size 1 1) (thickness 0.15)))
     )
@@
     (property "Sheetname" "")
     (attr through_hole)
-    (fp_text reference "Q5" (at 2.54 -3.56 90) (layer "F.SilkS")
+    (fp_text reference "Q5" (at 4.92 -2.29 90) (layer "F.SilkS")
       (effects (font (size 1 1) (thickness 0.15)))
     )
@@
     (property "Sheetname" "")
     (attr through_hole)
-    (fp_text reference "C1" (at 2.3 -3) (layer "F.SilkS")
+    (fp_text reference "C1" (at 2.42 -1.69) (layer "F.SilkS")
       (effects (font (size 1 1) (thickness 0.15)))
     )
@@
     (property "Sheetname" "")
     (attr through_hole)
-    (fp_text reference "Q2" (at 2.54 -3.56 90) (layer "F.SilkS")
+    (fp_text reference "Q2" (at 4.87 -2.45 90) (layer "F.SilkS")
       (effects (font (size 1 1) (thickness 0.15)))
     )
@@
     (property "Sheetname" "")
     (attr through_hole)
-    (fp_text reference "Q1" (at 2.54 -3.56 90) (layer "F.SilkS")
+    (fp_text reference "Q1" (at 4.95 -2.37 90) (layer "F.SilkS")
       (effects (font (size 1 1) (thickness 0.15)))
     )
@@
     (property "Sheetname" "")
     (attr through_hole)
-    (fp_text reference "FOCUS" (at -2.1 4.2 unlocked) (layer "F.SilkS")
+    (fp_text reference "FOCUS1" (at -2.1 4.2 unlocked) (layer "F.SilkS")
       (effects (font (size 1 1) (thickness 0.15)))
     )
@@
       (effects (font (size 1 1) (thickness 0.15)))
     )
-    (fp_text user "K" (at 0 -2.1 90) (layer "F.SilkS")
-      (effects (font (size 1 1) (thickness 0.15)))
-    )
     (fp_text user "K" (at 0 -2.1 90) (layer "F.Fab")
       (effects (font (size 1 1) (thickness 0.15)))
@@
     (property "Sheetname" "")
     (attr through_hole)
-    (fp_text reference "R34" (at 5.04 -5.8) (layer "F.SilkS")
+    (fp_text reference "R34" (at 4.78 -1.45) (layer "F.SilkS")
       (effects (font (size 1 1) (thickness 0.15)))
     )
@@
     (property "Sheetname" "")
     (attr through_hole)
-    (fp_text reference "ASTIG" (at -2.1 4.2 unlocked) (layer "F.SilkS")
+    (fp_text reference "ASTIG1" (at -2.1 4.2 unlocked) (layer "F.SilkS")
       (effects (font (size 1 1) (thickness 0.15)))
     )
@@
     (property "Sheetname" "")
     (attr through_hole)
-    (fp_text reference "INTENSITY" (at -2.1 4.2 unlocked) (layer "F.SilkS")
+    (fp_text reference "INTENSITY1" (at -2.1 4.2 unlocked) (layer "F.SilkS")
       (effects (font (size 1 1) (thickness 0.15)))
     )
@@
       (effects (font (size 1 1) (thickness 0.15)))
     )
-    (fp_text value "4.7K" (at 5.08 2.37 90) (layer "F.Fab")
+    (fp_text value "470K" (at 5.08 2.37 90) (layer "F.Fab")
       (effects (font (size 1 1) (thickness 0.15)))
     )
@@
     (property "Sheetname" "")
     (attr through_hole)
-    (fp_text reference "C18" (at 2.5 -6.25 90) (layer "F.SilkS")
+    (fp_text reference "C18" (at -1.095553 -5.22 180) (layer "F.SilkS")
       (effects (font (size 1 1) (thickness 0.15)))
     )
@@
     (property "Sheetname" "")
     (attr through_hole)
-    (fp_text reference "5V" (at 2.6 -0.2) (layer "F.SilkS")
+    (fp_text reference "5V1" (at 2.6 -0.2) (layer "F.SilkS")
       (effects (font (size 1 1) (thickness 0.15)))
     )
@@
     (property "Sheetname" "")
     (attr through_hole)
-    (fp_text reference "R47" (at 0.2 -2.4) (layer "F.SilkS")
+    (fp_text reference "R47" (at 4.64 -1.71) (layer "F.SilkS")
       (effects (font (size 1 1) (thickness 0.15)))
     )
@@
     (property "Sheetname" "")
     (attr through_hole)
-    (fp_text reference "U1" (at 3.81 -2.33) (layer "F.SilkS")
+    (fp_text reference "U1" (at 3.89 -1.49) (layer "F.SilkS")
       (effects (font (size 1 1) (thickness 0.15)))
     )
@@
     (property "Sheetname" "")
     (attr through_hole)
-    (fp_text reference "C16" (at 1.25 -5) (layer "F.SilkS")
+    (fp_text reference "C16" (at 4.711394 -3.54) (layer "F.SilkS")
       (effects (font (size 1 1) (thickness 0.15)))
     )
@@
     (property "Sheetname" "")
     (attr through_hole)
-    (fp_text reference "D5" (at 5.08 -2.47 90) (layer "F.SilkS")
+    (fp_text reference "D5" (at 4.71 2.04 90) (layer "F.SilkS")
       (effects (font (size 1 1) (thickness 0.15)))
     )
@@
       (effects (font (size 1 1) (thickness 0.15)))
     )
-    (fp_text user "K" (at 0 -2.1 90) (layer "F.SilkS")
-      (effects (font (size 1 1) (thickness 0.15)))
-    )
     (fp_text user "K" (at 0 -2.1 90) (layer "F.Fab")
       (effects (font (size 1 1) (thickness 0.15)))
@@
     (property "Sheetname" "")
     (attr through_hole)
-    (fp_text reference "Q4" (at 2.54 -3.56 90) (layer "F.SilkS")
+    (fp_text reference "Q4" (at 5.04 -2.25 90) (layer "F.SilkS")
       (effects (font (size 1 1) (thickness 0.15)))
     )
@@
     (property "Sheetname" "")
     (attr through_hole)
-    (fp_text reference "R4" (at 5.08 -2.37) (layer "F.SilkS")
+    (fp_text reference "R4" (at 5.26 -1.69) (layer "F.SilkS")
       (effects (font (size 1 1) (thickness 0.15)))
     )
@@
     (property "Sheetname" "")
     (attr through_hole)
-    (fp_text reference "C15" (at 2.5 -6.25) (layer "F.SilkS")
+    (fp_text reference "C15" (at 7.228385 -4.1) (layer "F.SilkS")
       (effects (font (size 1 1) (thickness 0.15)))
     )
@@
     (property "Sheetname" "")
     (attr through_hole)
-    (fp_text reference "YPOS" (at -2.1 4.2 unlocked) (layer "F.SilkS")
+    (fp_text reference "YPOS1" (at -2.1 4.2 unlocked) (layer "F.SilkS")
       (effects (font (size 1 1) (thickness 0.15)))
     )
@@
     (property "Sheetname" "")
     (attr through_hole)
-    (fp_text reference "R8" (at 5.08 -2.37) (layer "F.SilkS")
+    (fp_text reference "R8" (at 5.17 -1.7) (layer "F.SilkS")
       (effects (font (size 1 1) (thickness 0.15)))
     )
@@
     (property "Sheetname" "")
     (attr through_hole)
-    (fp_text reference "D3" (at 8.68 -2.2 90) (layer "F.SilkS")
+    (fp_text reference "D3" (at 5.43 -2.51 90) (layer "F.SilkS")
       (effects (font (size 1 1) (thickness 0.15)))
     )
@@
       (effects (font (size 1 1) (thickness 0.15)))
     )
-    (fp_text user "K" (at -1.72 1 90) (layer "F.SilkS")
-      (effects (font (size 1 1) (thickness 0.15)))
-    )
     (fp_text user "${REFERENCE}" (at 5.47 0 90) (layer "F.Fab")
       (effects (font (size 1 1) (thickness 0.15)))
@@
     (property "Sheetname" "")
     (attr through_hole)
-    (fp_text reference "C17" (at 4.838385 -5.96 90) (layer "F.SilkS")
+    (fp_text reference "C17" (at -1.361615 -5.06 180) (layer "F.SilkS")
       (effects (font (size 1 1) (thickness 0.15)))
     )
@@
     (property "Sheetname" "")
     (attr through_hole)
-    (fp_text reference "YSIZE" (at -2.1 4.2 unlocked) (layer "F.SilkS")
+    (fp_text reference "YSIZE1" (at -2.1 4.2 unlocked) (layer "F.SilkS")
       (effects (font (size 1 1) (thickness 0.15)))
     )
@@
     (property "Sheetname" "")
     (attr through_hole)
-    (fp_text reference "D4" (at 1.68 -5 90) (layer "F.SilkS")
+    (fp_text reference "D4" (at 4.25 -5.43 90) (layer "F.SilkS")
       (effects (font (size 1 1) (thickness 0.15)))
     )
@@
       (effects (font (size 1 1) (thickness 0.15)))
     )
-    (fp_text user "K" (at -2.12 1.2 90) (layer "F.SilkS")
-      (effects (font (size 1 1) (thickness 0.15)))
-    )
     (fp_text user "${REFERENCE}" (at 5.47 0 90) (layer "F.Fab")
       (effects (font (size 1 1) (thickness 0.15)))
@@
     (property "Sheetname" "")
     (attr through_hole)
-    (fp_text reference "R35" (at 5.08 -2.37) (layer "F.SilkS")
+    (fp_text reference "R35" (at 5.18 1.59) (layer "F.SilkS")
       (effects (font (size 1 1) (thickness 0.15)))
     )
@@
     (effects (font (size 1 1) (thickness 0.15)))
   )
-  (gr_text "CGULA\nCRT DRIVER \nREV. 1.0" (at 183.4 121.2) (layer "F.SilkS")
+  (gr_text "CGULA\nCRT DRIVER \nREV. 1.1" (at 183.4 121.2) (layer "F.SilkS")
     (effects (font (size 1 1) (thickness 0.15)))
   )
