File: CRT Main PCB/CRT Driver.kicad_sch (KiCad schematic)
At the start: 59 parts, among them J4 CRT, J5 TRANSFORMER, J6 XYZ SIGNAL IN, Q1 ZTX458, Q2 ZTX458, Q4 ZTX458, Q5 ZTX458, Q9 ZTX458, U1 TL082, U4 L78L05_TO92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

Commit message: PCB changes
Parts:
- removed U5: L79L05_SO8, Package_TO_SOT_THT:TO-92_Inline, symbol Regulator_Linear:L79L05_SO8
- added U5: L79L05_TO92, Package_TO_SOT_THT:TO-92_Inline_Wide, symbol Regulator_Linear:L79L05_TO92
- Q1, Q2, Q4, Q5, Q9, U4: footprint Package_TO_SOT_THT:TO-92_Inline -> Package_TO_SOT_THT:TO-92_Inline_Wide
Connections:
- net -5V: now also U5.3 (VO)
- net GND: now also U5.1 (GND)
- net at C22.2, D8.2 (A): now also U5.2 (VI)
Changed lines of the file:
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@@
       (effects (font (size 1.27 1.27)) (justify left))
     )
-    (property "Footprint" "Package_TO_SOT_THT:TO-92_Inline" (id 2) (at 238.76 43.815 0)
+    (property "Footprint" "Package_TO_SOT_THT:TO-92_Inline_Wide" (id 2) (at 238.76 43.815 0)
       (effects (font (size 1.27 1.27) italic) (justify left) hide)
     )
@@
       (effects (font (size 1.27 1.27)) (justify left))
     )
-    (property "Footprint" "Package_TO_SOT_THT:TO-92_Inline" (id 2) (at 219.71 122.555 0)
+    (property "Footprint" "Package_TO_SOT_THT:TO-92_Inline_Wide" (id 2) (at 219.71 122.555 0)
       (effects (font (size 1.27 1.27) italic) (justify left) hide)
     )
@@
     )
   )
+  (symbol (lib_id "Regulator_Linear:L79L05_TO92") (at 69.85 139.7 0) (unit 1)
+    (in_bom yes) (on_board yes) (fields_autoplaced)
+    (property "Reference" "U5" (id 0) (at 69.85 144.78 0))
+    (property "Value" "L79L05_TO92" (id 1) (at 69.85 147.32 0))
+    (property "Footprint" "Package_TO_SOT_THT:TO-92_Inline_Wide" (id 2) (at 69.85 144.78 0)
+      (effects (font (size 1.27 1.27) italic) hide)
+    )
+    (property "Datasheet" "http://www.farnell.com/datasheets/1827870.pdf" (id 3) (at 69.85 139.7 0)
+      (effects (font (size 1.27 1.27)) hide)
+    )
+    (pin "1")
+    (pin "2")
+    (pin "3")
+  )
   (symbol (lib_id "Regulator_Linear:L78L05_TO92") (at 69.85 111.76 0) (unit 1)
     (in_bom yes) (on_board yes) (fields_autoplaced)
     (property "Reference" "U4" (id 0) (at 69.85 104.14 0))
     (property "Value" "L78L05_TO92" (id 1) (at 69.85 106.68 0))
-    (property "Footprint" "Package_TO_SOT_THT:TO-92_Inline" (id 2) (at 69.85 106.045 0)
+    (property "Footprint" "Package_TO_SOT_THT:TO-92_Inline_Wide" (id 2) (at 69.85 106.045 0)
       (effects (font (size 1.27 1.27) italic) hide)
     )
@@
       (effects (font (size 1.27 1.27)) (justify left))
     )
-    (property "Footprint" "Package_TO_SOT_THT:TO-92_Inline" (id 2) (at 127 184.785 0)
+    (property "Footprint" "Package_TO_SOT_THT:TO-92_Inline_Wide" (id 2) (at 127 184.785 0)
       (effects (font (size 1.27 1.27) italic) (justify left) hide)
     )
@@
     (pin "2")
   )
-  (symbol (lib_id "Regulator_Linear:L79L05_SO8") (at 69.85 139.7 0) (unit 1)
-    (in_bom yes) (on_board yes) (fields_autoplaced)
-    (property "Reference" "U5" (id 0) (at 69.85 144.78 0))
-    (property "Value" "L79L05_SO8" (id 1) (at 69.85 147.32 0))
-    (property "Footprint" "Package_TO_SOT_THT:TO-92_Inline" (id 2) (at 69.85 144.78 0)
-      (effects (font (size 1.27 1.27) italic) hide)
-    )
-    (property "Datasheet" "http://www.farnell.com/datasheets/1827870.pdf" (id 3) (at 69.85 138.43 0)
-      (effects (font (size 1.27 1.27)) hide)
-    )
-    (pin "1")
-    (pin "2")
-    (pin "3")
-    (pin "4")
-    (pin "5")
-    (pin "6")
-    (pin "7")
-    (pin "8")
-  )
   (symbol (lib_id "Transistor_BJT:2N3904") (at 243.84 120.65 0) (mirror y) (unit 1)
     (in_bom yes) (on_board yes) (fields_autoplaced)
@@
       (effects (font (size 1.27 1.27)) (justify left))
     )
-    (property "Footprint" "Package_TO_SOT_THT:TO-92_Inline" (id 2) (at 238.76 122.555 0)
+    (property "Footprint" "Package_TO_SOT_THT:TO-92_Inline_Wide" (id 2) (at 238.76 122.555 0)
       (effects (font (size 1.27 1.27) italic) (justify left) hide)
     )
@@
       (effects (font (size 1.27 1.27)) (justify left))
     )
-    (property "Footprint" "Package_TO_SOT_THT:TO-92_Inline" (id 2) (at 219.71 43.815 0)
+    (property "Footprint" "Package_TO_SOT_THT:TO-92_Inline_Wide" (id 2) (at 219.71 43.815 0)
       (effects (font (size 1.27 1.27) italic) (justify left) hide)
     )
@@
     )
     (path "/7ed770b7-cb82-40f2-942f-896195512768"
-      (reference "Q1") (unit 1) (value "ZTX458") (footprint "Package_TO_SOT_THT:TO-92_Inline")
+      (reference "Q1") (unit 1) (value "ZTX458") (footprint "Package_TO_SOT_THT:TO-92_Inline_Wide")
     )
     (path "/ac414c2c-72a0-405f-a424-0697c03505a6"
-      (reference "Q2") (unit 1) (value "ZTX458") (footprint "Package_TO_SOT_THT:TO-92_Inline")
+      (reference "Q2") (unit 1) (value "ZTX458") (footprint "Package_TO_SOT_THT:TO-92_Inline_Wide")
     )
     (path "/c660bfba-9ae7-4b5b-a861-24815f5b8cb8"
-      (reference "Q4") (unit 1) (value "ZTX458") (footprint "Package_TO_SOT_THT:TO-92_Inline")
+      (reference "Q4") (unit 1) (value "ZTX458") (footprint "Package_TO_SOT_THT:TO-92_Inline_Wide")
     )
     (path "/6cba0056-3dc6-45c5-9992-466d2ccf8805"
-      (reference "Q5") (unit 1) (value "ZTX458") (footprint "Package_TO_SOT_THT:TO-92_Inline")
+      (reference "Q5") (unit 1) (value "ZTX458") (footprint "Package_TO_SOT_THT:TO-92_Inline_Wide")
     )
     (path "/9ee5c3e8-9357-4cf5-ada7-1cec35205c65"
-      (reference "Q9") (unit 1) (value "ZTX458") (footprint "Package_TO_SOT_THT:TO-92_Inline")
+      (reference "Q9") (unit 1) (value "ZTX458") (footprint "Package_TO_SOT_THT:TO-92_Inline_Wide")
     )
     (path "/5bcbcd82-c267-433b-8620-9bc6541c999f"
@@
     )
     (path "/8affa89d-ced8-4f87-95e4-2a816e736aa8"
-      (reference "U4") (unit 1) (value "L78L05_TO92") (footprint "Package_TO_SOT_THT:TO-92_Inline")
-    )
-    (path "/ab617da8-eeb3-4b72-b3b0-bf640e142ce7"
-      (reference "U5") (unit 1) (value "L79L05_SO8") (footprint "Package_TO_SOT_THT:TO-92_Inline")
+      (reference "U4") (unit 1) (value "L78L05_TO92") (footprint "Package_TO_SOT_THT:TO-92_Inline_Wide")
+    )
+    (path "/87d4ac54-7997-4874-9914-ce1ce295a6c1"
+      (reference "U5") (unit 1) (value "L79L05_TO92") (footprint "Package_TO_SOT_THT:TO-92_Inline_Wide")
     )
     (path "/6e79b566-dfa9-4433-9141-814835942bcf"

Commit message: fixed errors
Parts:
- R11: value 4.7K -> 470K
Changed lines of the file:
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@@
       (effects (font (size 1.27 1.27)) (justify right))
     )
-    (property "Value" "4.7K" (id 1) (at 81.28 74.9299 0)
+    (property "Value" "470K" (id 1) (at 81.28 74.9299 0)
       (effects (font (size 1.27 1.27)) (justify right))
     )
@@
     )
     (path "/1bf1093a-dae2-4c01-8a5c-60919479c7c6"
-      (reference "R11") (unit 1) (value "4.7K") (footprint "Resistor_THT:R_Axial_DIN0207_L6.3mm_D2.5mm_P10.16mm_Horizontal")
+      (reference "R11") (unit 1) (value "470K") (footprint "Resistor_THT:R_Axial_DIN0207_L6.3mm_D2.5mm_P10.16mm_Horizontal")
     )
     (path "/0c35cdc3-768e-4355-8303-76004a0f0766"
